File: pcb/SensEdu.kicad_sch (KiCad schematic)
At the start: 30 parts, among them J1 Power, J10 Barrel_Jack_Switch, J13 Conn_02x01, J14 Conn_02x01, J15 Conn_02x01, J16 Conn_02x01, J2 PWM, J3 Analog, J4 PWM, J5 Analog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

Commit message: pcb: New PCB revision (#88)
- Rearrange schematics
- Better symbols and footprints
- Better names and graphics
- Add simulations for DC offset after AC coupling
- Add BOM
- Redraw PCB layout
- Proper position for pressure and humidity sensor
- Better positions for EXT headers
- Silkscreen text labels for headers, pins, mics, etc.
- Change supply polarity and pin numbers of ADA4511
- Change cap of switches to 100n to reduce BOM
- Change supply of sensors to unison 3.3V
- Rearrange ADC pins
- Add digital switches instead of manual headers
- Add logos

---------

Co-authored-by: oberfeli <felix.ober@mailbox.org>
Parts:
- removed C3, C37, C38, C56: 10u, Capacitor_SMD:C_0805_2012Metric, symbol Device:C
- removed C36, C4, C55, C57, C8: 100n, Capacitor_SMD:C_0805_2012Metric, symbol Device:C
- removed C7: 1u, Capacitor_SMD:C_0805_2012Metric, symbol Device:C
- removed D1: LED, LED_SMD:LED_0805_2012Metric, symbol Device:LED
- removed FB1, FB2: FerriteBead, Inductor_SMD:L_1206_3216Metric, symbol Device:FerriteBead
- removed J10: Barrel_Jack_Switch, Connector_BarrelJack:BarrelJack_Wuerth_6941xx301002, symbol Connector:Barrel_Jack_Switch
- removed J13, J14, J15, J16: Conn_02x01, Connector_PinSocket_2.54mm:PinSocket_1x02_P2.54mm_Vertical, symbol Connector_Generic:Conn_02x01
- removed JP3: Jumper_3_Bridged12, Connector_PinHeader_2.54mm:PinHeader_1x03_P2.54mm_Vertical, symbol Jumper:Jumper_3_Bridged12
- removed R1: 47, Resistor_SMD:R_0805_2012Metric, symbol Device:R
- removed U12: TLS850C2TE_V33, Package_TO_SOT_SMD:TO-252-4, symbol SensEdu:TLS850C2TEV50ATMA1
- removed U13: NCP1117-2.5_SOT223, Package_TO_SOT_SMD:SOT-223-3_TabPin2, symbol Regulator_Linear:NCP1117-2.5_SOT223
- removed U3: LT1790ACS6-1.25, Package_TO_SOT_SMD:TSOT-23-6, symbol SensEdu:LT1790-2.5_sensedu
- J1, J3, J4, J5, J6: symbol Connector_Generic:Conn_01x08 -> SensEdu:Conn_01x08
- J2: symbol Connector_Generic:Conn_01x10 -> SensEdu:Conn_01x10
- J7: symbol Connector_Generic:Conn_02x18_Odd_Even -> SensEdu:Conn_02x18_Odd_Even; now not fitted
Connections:
- net *2 renamed 3*
- net *3 renamed 4*
- net *4 renamed SE_PWM_1
- net *6 renamed S1
- net *7 renamed S2
- net 37 renamed SE_PWM_2
- net 3V3 renamed 3V3_INO
- net 48 renamed SE_PWM_3
- net 5V0 renamed +5V_ARDUINO
- net A0 renamed MIC1_OUT
- net A1 renamed MIC2_OUT
- net A10 renamed AMP3_OUT
- net A12 renamed DAC0
- net A13 renamed DAC1
- net A2 renamed MIC3_OUT
- net A3 renamed MIC4_OUT
- net A5: no longer names the net of J3.6 (Pin_6)
- net A6: no longer names the net of J3.7 (Pin_7)
- net A7: no longer names the net of J3.8 (Pin_8)
- net A8 renamed AMP1_OUT
- net A9 renamed AMP2_OUT
- net Microphones/MIC7_OUT renamed AMP4_OUT
- net SCL/21 renamed SCL
- net SDA/20 renamed SDA
- no-connect marks 69 -> 59
Other:
- sheet Pressure Sensor renamed Sensors
- added sheet Power (power.kicad_sch)
- sheet Microphones ports: added AMP1_EXT_OUT, AMP2_EXT_OUT, AMP3_EXT_OUT, AMP4_EXT_OUT; removed MIC5_OUT, MIC6_OUT, MIC7_OUT, MIC8_OUT
- sheet Sensors: file Pressure_sensor.kicad_sch -> Sensors.kicad_sch
- sheet Sensors ports: added SCL, SDA; removed SCL1, SDA1
- sheet Speakers ports: added none; removed PWM_2, PWM_3
- note removed: "LOW DROPOUT VOLTAGE REFERENCE 3.3V->1.25V"
- note removed: "POWER"
- title: SensEdu 0.7 -> SensEdu
- moved on the sheet: J1, J2, J3, J4, J5, J6
